Commit message: Solved third exercise with a few problems

File: src/my_r2d2/urdf/r2d2.urdf (robot description, URDF)
Before this commit: robot macroed, 17 links, 16 joints
Links:
- removed link lense
- added link base_footprint
- added link lense_testing, mass 0.5; collision sphere radius=0.038; visual sphere radius=0.038
Joints:
- added joint base_footprintToLink: type fixed, parent base_link, child base_footprint, origin xyz=0 0 -0.47
- joint tolense: child lense -> lense_testing

File: src/my_r2d2/urdf/r2d2.xacro (robot description, xacro)
@@ -214,23 +214,33 @@
     <origin xyz="${.707*width+0.04} 0 ${.707*width}"/>
   </joint>
-  <link name="lense">
-    <visual>
-      <geometry>
-        <sphere radius="0.038"/>
-      </geometry>
-      <material name="black"/>
+  <xacro:macro name="lense" params="material baselen name mass">
+  <link name="${name}">
+    <visual>
+      <geometry>
+        <sphere radius="${baselen}"/>
+      </geometry>
+      <material name="${material}"/>
       <origin xyz="-0.015 0 0"/>
     </visual>
     <collision>
       <geometry>
-        <sphere radius="0.038"/>
+        <sphere radius="${baselen}"/>
       </geometry>
       <origin xyz="-0.015 0 0"/>
     </collision>
-    <xacro:default_inertial mass="0.5"/>
+    <xacro:default_inertial mass="${mass}"/>
   </link>
   <joint name="tolense" type="fixed">
     <parent link="box"/>
-    <child link="lense"/>
+    <child link="${name}"/>
+  </joint>
+  </xacro:macro>
+  <xacro:lense material="black" baselen="0.038" name="lense_testing" mass="0.5"/>
+  <link name="base_footprint">-
+  </link>
+  <joint name="base_footprintToLink" type="fixed">
+    <parent link="base_link"/>
+    <child link="base_footprint"/>
+    <origin xyz="0 0 -${bodylen/2 + 0.1 + wheeldiam}"/>
   </joint>
 </robot>

Commit message: Fixed error, joints were opposite

File: src/my_r2d2/urdf/r2d2.urdf (robot description, URDF)
Before this commit: robot macroed, 18 links, 17 joints
Joints:
- joint base_footprintToLink: child base_footprint -> base_link; origin xyz=0 0 -0.47 -> xyz=0 0 0.47; parent base_link -> base_footprint

File: src/my_r2d2/urdf/r2d2.xacro (robot description, xacro)
@@ -240,7 +240,7 @@
   </link>
   <joint name="base_footprintToLink" type="fixed">
-    <parent link="base_link"/>
-    <child link="base_footprint"/>
-    <origin xyz="0 0 -${bodylen/2 + 0.1 + wheeldiam}"/>
+    <parent link="base_footprint"/>
+    <origin xyz="0 0 ${bodylen/2 + 0.1 + wheeldiam}"/>
+    <child link="base_link"/>
   </joint>
 </robot>

Commit message: ex4

File: src/my_r2d2/urdf/r2d2.urdf (robot description, URDF)
Before this commit: robot macroed, 18 links, 17 joints
Links:
- removed link lense_testing
- added link lense, mass 0.5; collision sphere radius=0.038; visual sphere radius=0.038
Joints:
- joint tolense: child lense_testing -> lense

File: src/my_r2d2/urdf/r2d2.xacro (robot description, xacro)
@@ -236,5 +236,5 @@
   </joint>
   </xacro:macro>
-  <xacro:lense material="black" baselen="0.038" name="lense_testing" mass="0.5"/>
+  <xacro:lense material="black" baselen="0.038" name="lense" mass="0.5"/>
   <link name="base_footprint">-
   </link>
@@ -244,3 +244,10 @@
     <child link="base_link"/>
   </joint>
+  <link name="eye">
+  </link>
+  <joint name="eyeToLense" type="fixed">
+    <parent link="lense"/>
+    <origin xyz="0.1 0 0" rpy="-${pi/2} ${pi/2*4} -${pi/2}"/>
+    <child link="eye"/>
+  </joint>
 </robot>
